Commit message: Add local-box scenario, Cosmetic changes in scripts

File: urdf/object.urdf (robot description, URDF)
Before this commit: robot object, 3 links, 2 joints
Links:
- link base_link: mass None -> 1.0
Joints:
- joint j_translation_x: limit lower=-5 upper=5 effort=1.0 velocity=1.0 -> lower=-100 upper=100 effort=1.0 velocity=1.0
- joint j_translation_y: limit lower=-5 upper=5 effort=1.0 velocity=1.0 -> lower=-2 upper=2 effort=1.0 velocity=1.0
