Commit message: Some path-optim updates, New parabola files

File: urdf/large_object.urdf (robot description, URDF)
Before this commit: robot object, 3 links, 2 joints
Links:
- link true_base_link: geometry collision cylinder length=0.8 radius=0.14; visual cylinder length=0.8 radius=0.14
Joints:
- joint j_translation_x: limit lower=-8 upper=8 effort=1.0 velocity=1.0 -> lower=-4 upper=13 effort=1.0 velocity=1.0
- joint j_translation_y: limit lower=-3 upper=5 effort=1.0 velocity=1.0 -> lower=-6 upper=6 effort=1.0 velocity=1.0
