Commit message: Update matplotlib tools to orthogonal-collision-constraints

File: urdf/cylinder_obstacle.urdf (robot description, URDF)
Before this commit: robot cylinder_obstacle, 1 links, 0 joints
Links:
- added link l_second_cylinder; collision cylinder length=0.4 radius=1.; visual cylinder length=0.4 radius=1.
- link obstacle_base: mass 1.0 -> None
Joints:
- added joint j_second_cylinder: type fixed, parent obstacle_base, child l_second_cylinder, origin xyz=0 0 0 rpy=0 0 0
